Commit message: Modification parameters

File: dr_description/urdf/yumi_main.xacro (robot description, xacro)
@@ -5,5 +5,5 @@
   <xacro:arg name="table" default="false"/>
   <xacro:arg name="camera" default="false"/>
-  <xacro:arg name="arms_hw_interface" default="VelocityJointInterface"/>
+  <xacro:arg name="arms_hw_interface" default="PositionJointInterface"/>
   <xacro:arg name="grippers_hw_interface" default="EffortJointInterface"/>
   <!-- ******************************************** -->

File: yumi_description/urdf/yumi_main.xacro (robot description, xacro)
@@ -4,5 +4,5 @@
   <xacro:arg name="table" default="false"/>
   <xacro:arg name="camera" default="false"/>
-  <xacro:arg name="arms_hw_interface" default="VelocityJointInterface"/>
+  <xacro:arg name="arms_hw_interface" default="PositionJointInterface"/>
   <xacro:arg name="smart_gripper" default="false"/>
   <xacro:arg name="grippers_hw_interface" default="EffortJointInterface"/>
@@ -16,7 +16,7 @@
   <!--Import the yumi macro                         -->
   <xacro:include filename="$(find yumi_description)/urdf/yumi.xacro"/>
-  <link name="world"/>
-  <joint name="world_joint" type="fixed">
-    <parent link="world"/>
+  <link name="${yumi_parent}"/>
+  <joint name="${yumi_parent}_joint" type="fixed">
+    <parent link="${yumi_parent}"/>
     <child link="yumi_base_link"/>
     <origin xyz="0 0 0.1" rpy="0 0 0" />
